Commit message: add gazebo

File: lookso_jr_description/urdf/lookso_jr.gazebo.xacro (robot description, xacro)
@@ -11,10 +11,4 @@
   <gazebo reference="world">
   </gazebo>
-  <!-- Base -->
-<!--  <gazebo reference="base">
-    <mu1>0.2</mu1>
-    <mu2>0.2</mu2>
-    <material>Gazebo/Grey</material>
-  </gazebo>-->
   <!-- Link1 -->
   <gazebo reference="link1">
@@ -41,3 +35,9 @@
     <material>Gazebo/Grey</material>
   </gazebo>
+  <!-- Link4 -->
+  <gazebo reference="link5">
+    <mu1>0.2</mu1>
+    <mu2>0.2</mu2>
+    <material>Gazebo/Grey</material>
+  </gazebo>
 </robot>

File: lookso_jr_description/urdf/lookso_jr.xacro (robot description, xacro)
@@ -5,5 +5,5 @@
   <xacro:property name="pi" value="3.141592654" />
   <!-- Import all Gazebo-customization elements, including Gazebo colors -->
-<!--  <xacro:include filename="$(find lookso_jr_description)/urdf/open_manipulator_chain.gazebo" />-->
+  <xacro:include filename="$(find lookso_jr_description)/urdf/lookso_jr.gazebo.xacro" />
   <!-- Import Rviz colors -->
   <xacro:include filename="$(find lookso_jr_description)/urdf/materials.xacro" />

Commit message: update

File: lookso_jr_description/urdf/lookso_jr.gazebo.xacro (robot description, xacro)
@@ -41,3 +41,43 @@
     <material>Gazebo/Grey</material>
   </gazebo>
+  <transmission name="tran1">
+    <type>transmission_interface/SimpleTransmission</type>
+    <joint name="joint1">
+      <hardwareInterface>PositionJointInterface</hardwareInterface>
+    </joint>
+    <actuator name="motor1">
+      <hardwareInterface>PositionJointInterface</hardwareInterface>
+      <mechanicalReduction>1</mechanicalReduction>
+    </actuator>
+  </transmission>
+  <transmission name="tran2">
+    <type>transmission_interface/SimpleTransmission</type>
+    <joint name="joint2">
+      <hardwareInterface>PositionJointInterface</hardwareInterface>
+    </joint>
+    <actuator name="motor2">
+      <hardwareInterface>PositionJointInterface</hardwareInterface>
+      <mechanicalReduction>1</mechanicalReduction>
+    </actuator>
+  </transmission>
+  <transmission name="tran3">
+    <type>transmission_interface/SimpleTransmission</type>
+    <joint name="joint3">
+      <hardwareInterface>PositionJointInterface</hardwareInterface>
+    </joint>
+    <actuator name="motor3">
+      <hardwareInterface>PositionJointInterface</hardwareInterface>
+      <mechanicalReduction>1</mechanicalReduction>
+    </actuator>
+  </transmission>
+  <transmission name="tran4">
+    <type>transmission_interface/SimpleTransmission</type>
+    <joint name="joint4">
+      <hardwareInterface>PositionJointInterface</hardwareInterface>
+    </joint>
+    <actuator name="motor4">
+      <hardwareInterface>PositionJointInterface</hardwareInterface>
+      <mechanicalReduction>1</mechanicalReduction>
+    </actuator>
+  </transmission>
 </robot>

File: lookso_jr_description/urdf/lookso_jr.xacro (robot description, xacro)
@@ -12,5 +12,5 @@
   </link>
   <!-- World fixed joint-->
-  <joint name="world_fixed" type="fixed">
+  <joint name="world_fixed" type="floating">
     <origin xyz="0 0 0" rpy="0 0 0"/>
     <parent link="world"/>
@@ -34,8 +34,8 @@
     <inertial>
       <origin xyz="0 0 0" />
-      <mass value="0.01" />
-      <inertia ixx="0.001" ixy="0.0" ixz="0.0"
-               iyy="0.001" iyz="0.0"
-               izz="0.001" />
+      <mass value="${0.1*100}" />
+      <inertia ixx="1.0" ixy="0.0" ixz="0.0"
+               iyy="1.0" iyz="0.0"
+               izz="1.0" />
     </inertial>
   </link>
@@ -49,17 +49,8 @@
     <dynamics damping="0.1"/>
   </joint>
-  <transmission name="tran1">
-    <type>transmission_interface/SimpleTransmission</type>
-    <joint name="joint1">
-      <hardwareInterface>PositionJointInterface</hardwareInterface>
-    </joint>
-    <actuator name="motor1">
-      <hardwareInterface>PositionJointInterface</hardwareInterface>
-      <mechanicalReduction>1</mechanicalReduction>
-    </actuator>
-  </transmission>
+  <!-- Link 2 -->
   <link name="link2">
     <collision>
-      <origin xyz="0.0 0.0 0.0" rpy="0 0 0"/>
+      <origin xyz="0.0 0.0 -0.054" rpy="0 0 0"/>
       <geometry>
         <mesh filename="package://lookso_jr_description/meshes/link2.stl" scale="0.001 0.001 0.001"/>
@@ -75,10 +66,11 @@
     <inertial>
       <origin xyz="0 0 0" />
-      <mass value="0.01" />
-      <inertia ixx="0.001" ixy="0.0" ixz="0.0"
-               iyy="0.001" iyz="0.0"
-               izz="0.001" />
+      <mass value="0.4" />
+      <inertia ixx="1.0" ixy="0.0" ixz="0.0"
+               iyy="1.0" iyz="0.0"
+               izz="1.0" />
     </inertial>
   </link>
+  <!-- Joint 2 -->
   <joint name="joint2" type="revolute">
     <parent link="link2"/>
@@ -89,17 +81,8 @@
     <dynamics damping="0.1"/>
   </joint>
-  <transmission name="tran2">
-    <type>transmission_interface/SimpleTransmission</type>
-    <joint name="joint2">
-      <hardwareInterface>PositionJointInterface</hardwareInterface>
-    </joint>
-    <actuator name="motor2">
-      <hardwareInterface>PositionJointInterface</hardwareInterface>
-      <mechanicalReduction>1</mechanicalReduction>
-    </actuator>
-  </transmission>
+  <!-- Link 3 -->
   <link name="link3">
     <collision>
-      <origin xyz="0 0 0" rpy="0 0 0"/>
+      <origin xyz="0.0263 0.0 -0.1198" rpy="0 0 0"/>
       <geometry>
         <mesh filename="package://lookso_jr_description/meshes/link3.stl" scale="0.001 0.001 0.001"/>
@@ -115,10 +98,11 @@
     <inertial>
       <origin xyz="0 0 0" />
-      <mass value="0.01" />
-      <inertia ixx="0.001" ixy="0.0" ixz="0.0"
-               iyy="0.001" iyz="0.0"
-               izz="0.001" />
+      <mass value="${0.05*100}" />
+      <inertia ixx="1.0" ixy="0.0" ixz="0.0"
+               iyy="1.0" iyz="0.0"
+               izz="1.0" />
     </inertial>
   </link>
+  <!-- Joint 3 -->
   <joint name="joint3" type="revolute">
     <parent link="link3"/>
@@ -129,17 +113,8 @@
     <dynamics damping="0.1"/>
   </joint>
-  <transmission name="tran3">
-    <type>transmission_interface/SimpleTransmission</type>
-    <joint name="joint3">
-      <hardwareInterface>PositionJointInterface</hardwareInterface>
-    </joint>
-    <actuator name="motor3">
-      <hardwareInterface>PositionJointInterface</hardwareInterface>
-      <mechanicalReduction>1</mechanicalReduction>
-    </actuator>
-  </transmission>
+  <!-- Link 4 -->
   <link name="link4">
     <collision>
-      <origin xyz="0 0 0.0" rpy="0 0 0"/>
+      <origin xyz="0.0263 0.0 -0.1948" rpy="0 0 0"/>
       <geometry>
         <mesh filename="package://lookso_jr_description/meshes/link4.stl" scale="0.001 0.001 0.001"/>
@@ -155,10 +130,11 @@
     <inertial>
       <origin xyz="0 0 0" />
-      <mass value="0.01" />
-      <inertia ixx="0.001" ixy="0.0" ixz="0.0"
-               iyy="0.001" iyz="0.0"
-               izz="0.001" />
+      <mass value="${0.2*100}" />
+      <inertia ixx="1.0" ixy="0.0" ixz="0.0"
+               iyy="1.0" iyz="0.0"
+               izz="1.0" />
     </inertial>
   </link>
+  <!-- Joint 4 -->
   <joint name="joint4" type="revolute">
     <parent link="link4"/>
@@ -169,17 +145,7 @@
     <dynamics damping="0.1"/>
   </joint>
-  <transmission name="tran4">
-    <type>transmission_interface/SimpleTransmission</type>
-    <joint name="joint4">
-      <hardwareInterface>PositionJointInterface</hardwareInterface>
-    </joint>
-    <actuator name="motor4">
-      <hardwareInterface>PositionJointInterface</hardwareInterface>
-      <mechanicalReduction>1</mechanicalReduction>
-    </actuator>
-  </transmission>
   <link name="link5">
     <collision>
-      <origin xyz="0 0 0.0" rpy="0 0 0"/>
+      <origin xyz="0.0143 0.0 -0.2321" rpy="0 0 0"/>
       <geometry>
         <mesh filename="package://lookso_jr_description/meshes/link5.stl" scale="0.001 0.001 0.001"/>
@@ -194,9 +160,9 @@
     </visual>
     <inertial>
-      <origin xyz="0 0 0" />
-      <mass value="0.01" />
-      <inertia ixx="0.001" ixy="0.0" ixz="0.0"
-               iyy="0.001" iyz="0.0"
-               izz="0.001" />
+      <origin xyz="0.075 0 0.050" />
+      <mass value="${0.7*100}" />
+      <inertia ixx="1.0" ixy="0.0" ixz="0.0"
+               iyy="1.0" iyz="0.0"
+               izz="1.0" />
     </inertial>
   </link>
