Commit message: update mesh file

File: lookso_jr_description/urdf/lookso_jr.xacro (robot description, xacro)
@@ -13,5 +13,5 @@
   <!-- World fixed joint-->
   <joint name="world_fixed" type="fixed">
-    <origin xyz="0 0 0" rpy="1.57 0 0"/>
+    <origin xyz="0 0 0" rpy="0 0 0"/>
     <parent link="world"/>
     <child link="link1"/>
@@ -33,8 +33,9 @@
     </visual>
     <inertial>
-      <origin xyz="0.00025 0.00000 0.01780" rpy="0 0 0"/>
-      <mass value="0.087"/>
-      <inertia ixx="1.0" ixy="0.0" ixz="0.0" iyy="1.0" iyz="0.0" izz="1.0" />
-      <inertia ixx="0.00001378" ixy="0.0" ixz="-0.00000025" iyy="0.00002381" iyz="0.0" izz="0.00002107" />
+      <origin xyz="0 0 0" />
+      <mass value="0.01" />
+      <inertia ixx="0.001" ixy="0.0" ixz="0.0"
+               iyy="0.001" iyz="0.0"
+               izz="0.001" />
     </inertial>
   </link>
@@ -43,5 +44,5 @@
     <parent link="link1"/>
     <child link="link2"/>
-    <origin xyz="0.0 0.0 0.010" rpy="0 0 0"/>
+    <origin xyz="0.0 0.0 0.0" rpy="0 0 0"/>
     <axis xyz="0 0 1"/>
     <limit velocity="6.5" effort="1000" lower="${-pi*0.9}" upper="${pi*0.9}" />
@@ -73,8 +74,9 @@
     </visual>
     <inertial>
-      <origin xyz="0.00002 -0.00045 0.03293" rpy="0 0 0"/>
-      <mass value="0.117"/>
-      <inertia ixx="1.0" ixy="0.0" ixz="0.0" iyy="1.0" iyz="0.0" izz="1.0" />
-      <inertia ixx="0.00004110" ixy="0.0" ixz="-0.00000025" iyy="0.00002381" iyz="0.0" izz="0.00002107" />
+      <origin xyz="0 0 0" />
+      <mass value="0.01" />
+      <inertia ixx="0.001" ixy="0.0" ixz="0.0"
+               iyy="0.001" iyz="0.0"
+               izz="0.001" />
     </inertial>
   </link>
@@ -112,8 +114,9 @@
     </visual>
     <inertial>
-      <origin xyz="0.00966 -0.00034 0.11795" rpy="0 0 0"/>
-      <mass value="0.156"/>
-      <inertia ixx="1.0" ixy="0.0" ixz="0.0" iyy="1.0" iyz="0.0" izz="1.0" />
-      <inertia ixx="0.00041624" ixy="0.00000017" ixz="-0.00004492" iyy="0.00042758" iyz="0.00000159" izz="0.00005317" />
+      <origin xyz="0 0 0" />
+      <mass value="0.01" />
+      <inertia ixx="0.001" ixy="0.0" ixz="0.0"
+               iyy="0.001" iyz="0.0"
+               izz="0.001" />
     </inertial>
   </link>
@@ -151,8 +154,9 @@
     </visual>
     <inertial>
-      <origin xyz="0.11076 -0.00035 0.00050" rpy="0 0 0"/>
-      <mass value="0.149"/>
-      <inertia ixx="1.0" ixy="0.0" ixz="0.0" iyy="1.0" iyz="0.0" izz="1.0" />
-      <inertia ixx="0.00003083" ixy="0.00000147" ixz="-0.00000222" iyy="0.00036703" iyz="-0.00000003" izz="0.00037667" />
+      <origin xyz="0 0 0" />
+      <mass value="0.01" />
+      <inertia ixx="0.001" ixy="0.0" ixz="0.0"
+               iyy="0.001" iyz="0.0"
+               izz="0.001" />
     </inertial>
   </link>
@@ -175,4 +179,25 @@
     </actuator>
   </transmission>
-<link name="link5"/>
+  <link name="link5">
+    <collision>
+      <origin xyz="0 0 0.0" rpy="0 0 0"/>
+      <geometry>
+        <mesh filename="package://lookso_jr_description/meshes/link5.stl" scale="0.001 0.001 0.001"/>
+      </geometry>
+    </collision>
+    <visual>
+      <origin xyz="0.0 0 0.0" rpy="0 0 0"/>
+      <geometry>
+        <mesh filename="package://lookso_jr_description/meshes/link5.stl" scale="0.001 0.001 0.001"/>
+      </geometry>
+      <material name="grey"/>
+    </visual>
+    <inertial>
+      <origin xyz="0 0 0" />
+      <mass value="0.01" />
+      <inertia ixx="0.001" ixy="0.0" ixz="0.0"
+               iyy="0.001" iyz="0.0"
+               izz="0.001" />
+    </inertial>
+  </link>
 </robot>

Commit message: modify urdf

File: lookso_jr_description/urdf/lookso_jr.xacro (robot description, xacro)
@@ -44,5 +44,5 @@
     <parent link="link1"/>
     <child link="link2"/>
-    <origin xyz="0.0 0.0 0.0" rpy="0 0 0"/>
+    <origin xyz="0.0 0.0 0.054" rpy="0 0 0"/>
     <axis xyz="0 0 1"/>
     <limit velocity="6.5" effort="1000" lower="${-pi*0.9}" upper="${pi*0.9}" />
@@ -67,5 +67,5 @@
     </collision>
     <visual>
-      <origin xyz="0.0 0.0 0.00" rpy="0 0 0"/>
+      <origin xyz="0.0 0.0 -0.054" rpy="0 0 0"/>
       <geometry>
         <mesh filename="package://lookso_jr_description/meshes/link2.stl" scale="0.001 0.001 0.001"/>
@@ -84,5 +84,5 @@
     <parent link="link2"/>
     <child link="link3"/>
-    <origin xyz="0.0 0.0 0.0" rpy="0 0 0"/>
+    <origin xyz="-0.0263 0.0 0.0658" rpy="0 0 0"/>
     <axis xyz="0 1 0"/>
     <limit velocity="6.5" effort="1000" lower="${-pi*0.9}" upper="${pi*0.9}" />
@@ -107,5 +107,5 @@
     </collision>
     <visual>
-      <origin xyz="0.0 0 0.0" rpy="0 0 0"/>
+      <origin xyz="0.0263 0.0 -0.1198" rpy="0 0 0"/>
       <geometry>
         <mesh filename="package://lookso_jr_description/meshes/link3.stl" scale="0.001 0.001 0.001"/>
@@ -124,5 +124,5 @@
     <parent link="link3"/>
     <child link="link4"/>
-    <origin xyz="0.0 0 0.0" rpy="0 0 0"/>
+    <origin xyz="0.0 0 0.075" rpy="0 0 0"/>
     <axis xyz="0 1 0"/>
     <limit velocity="6.5" effort="1000" lower="${-pi*0.9}" upper="${pi*0.9}" />
@@ -147,5 +147,5 @@
     </collision>
     <visual>
-      <origin xyz="0.0 0 0.0" rpy="0 0 0"/>
+      <origin xyz="0.0263 0.0 -0.1948" rpy="0 0 0"/>
       <geometry>
         <mesh filename="package://lookso_jr_description/meshes/link4.stl" scale="0.001 0.001 0.001"/>
@@ -164,5 +164,5 @@
     <parent link="link4"/>
     <child link="link5"/>
-    <origin xyz="0.0 0.0 0.0" rpy="0 0 0"/>
+    <origin xyz="0.012 0.0 0.0373" rpy="0 0 0"/>
     <axis xyz="0 0 1"/>
     <limit velocity="6.5" effort="1000" lower="${-pi*0.9}" upper="${pi*0.9}" />
@@ -187,5 +187,5 @@
     </collision>
     <visual>
-      <origin xyz="0.0 0 0.0" rpy="0 0 0"/>
+      <origin xyz="0.0143 0.0 -0.2321" rpy="0 0 0"/>
       <geometry>
         <mesh filename="package://lookso_jr_description/meshes/link5.stl" scale="0.001 0.001 0.001"/>

Commit message: add moveit

File: lookso_jr_description/urdf/lookso_jr.xacro (robot description, xacro)
@@ -12,5 +12,5 @@
   </link>
   <!-- World fixed joint-->
-  <joint name="world_fixed" type="floating">
+  <joint name="world_fixed" type="fixed">
     <origin xyz="0 0 0" rpy="0 0 0"/>
     <parent link="world"/>
